File: D1MiniChainCounterWLAN.kicad_pcb (KiCad board)
At the start: 2 copper layers, 74.9 x 50.2 mm, 20 parts, among them J1 Power, J2 D24V10F5, J3 Chain Sens., J4 Chain Sw., K1 FINDER-32.21-x300, K2 FINDER-32.21-x300, Q1 BC337, Q2 BC337, Q3 BC337, Q4 BC337, U1 WeMos_D1_mini, U2 H11L1

Commit message: Add files via upload
Other:
- board text added: "Chain Counter WLAN Rev 1.0"
Changed lines of the file:
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@@
   (general
     (thickness 1.6)
-    (drawings 14)
+    (drawings 15)
     (tracks 183)
     (zones 0)
@@
     )
   )
+  (gr_text "Chain Counter\nWLAN\nRev 1.0" (at 107.315 59.055) (layer F.SilkS)
+    (effects (font (size 1.5 1.5) (thickness 0.3)))
+  )
   (gr_line (start 96.52 95.25) (end 96.52 81.28) (layer F.SilkS) (width 0.15))

Commit message: Add files via upload
Parts:
- K1, K2: value FINDER-32.21-x300 -> G5Q-1A; footprint Relay_THT:Relay_SPST_Finder_32.21-x300 -> Relay_THT:Relay_SPST_Omron-G5Q-1A
Connections:
- net Net-(J1-Pad2) renamed GND
- D1 pad 2: Net-(D1-Pad2) -> +12V
- D2 pad 1: Net-(D2-Pad1) -> +5V
- D3 pad 1: Net-(D2-Pad1) -> +5V
- J1 pad 1: Net-(D1-Pad2) -> +12V
- J2 pad 1: (no net) -> Net-(J2-Pad1)
- J2 pad 2: (no net) -> Net-(J2-Pad2)
- J2 pad 5: Net-(D2-Pad1) -> +5V
- R1 pad 1: Net-(D1-Pad2) -> +12V
- U1 pad 1: (no net) -> Net-(U1-Pad1)
- U1 pad 15: (no net) -> Net-(U1-Pad15)
- U1 pad 16: (no net) -> Net-(U1-Pad16)
- U1 pad 2: (no net) -> Net-(U1-Pad2)
- U1 pad 3: (no net) -> Net-(U1-Pad3)
- U1 pad 5: (no net) -> Net-(U1-Pad5)
- U1 pad 6: (no net) -> Net-(U1-Pad6)
- U1 pad 7: (no net) -> Net-(U1-Pad7)
- U1 pad 8: (no net) -> Net-(U1-Pad8)
- U1 pad 9: Net-(D2-Pad1) -> +5V
- U2 pad 3: (no net) -> Net-(U2-Pad3)
- U2 pad 6: Net-(D2-Pad1) -> +5V
Routing:
- net +5V: track 0.00 -> 195.6 mm, vias 0 -> 2
- net Net-(D2-Pad1): track 172.3 -> 0.00 mm
- net Net-(D1-Pad2): track 92.2 -> 0.00 mm, vias 2 -> 0
- net +12V: track 0.00 -> 92.2 mm, vias 0 -> 2
- net Net-(D2-Pad2): track 29.8 -> 38.3 mm, vias 1 -> 2
- net Net-(D3-Pad2): track 21.8 -> 17.9 mm

Commit message: Add files via upload
Routing:
- net +5V: track 195.6 -> 168.3 mm, vias 2 -> 4
Changed lines of the file:
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@@
     (thickness 1.6)
     (drawings 15)
-    (tracks 197)
+    (tracks 201)
     (zones 0)
     (modules 20)
@@
   (segment (start 140.335 95.25) (end 137.16 95.25) (width 0.25) (layer B.Cu) (net 2))
   (segment (start 140.97 94.615) (end 140.335 95.25) (width 0.25) (layer B.Cu) (net 2))
-  (segment (start 105.41 74.93) (end 105.41 80.01) (width 0.25) (layer B.Cu) (net 17))
-  (segment (start 144.78 80.645) (end 144.78 82.55) (width 0.25) (layer B.Cu) (net 17))
-  (segment (start 135.255 80.01) (end 144.145 80.01) (width 0.25) (layer B.Cu) (net 17))
-  (segment (start 144.145 80.01) (end 144.78 80.645) (width 0.25) (layer B.Cu) (net 17))
-  (segment (start 136.525 52.07) (end 137.424999 52.969999) (width 0.25) (layer B.Cu) (net 17))
   (segment (start 144.145 60.96) (end 144.145 64.77) (width 0.25) (layer B.Cu) (net 3))
   (segment (start 144.78 65.405) (end 144.145 64.77) (width 0.25) (layer B.Cu) (net 3))
@@
   (segment (start 151.13 64.135) (end 146.685 59.69) (width 0.25) (layer F.Cu) (net 16))
   (segment (start 151.13 87.63) (end 151.13 64.135) (width 0.25) (layer F.Cu) (net 16))
+  (segment (start 105.41 74.93) (end 105.41 80.01) (width 0.25) (layer B.Cu) (net 17))
+  (segment (start 144.78 80.645) (end 144.78 82.55) (width 0.25) (layer B.Cu) (net 17))
+  (segment (start 135.255 80.01) (end 144.145 80.01) (width 0.25) (layer B.Cu) (net 17))
+  (segment (start 144.145 80.01) (end 144.78 80.645) (width 0.25) (layer B.Cu) (net 17))
+  (segment (start 136.525 52.07) (end 137.424999 52.969999) (width 0.25) (layer B.Cu) (net 17))
   (segment (start 97.79 74.93) (end 105.41 74.93) (width 0.25) (layer B.Cu) (net 17))
   (segment (start 96.52 76.2) (end 97.79 74.93) (width 0.25) (layer B.Cu) (net 17))
@@
   (segment (start 146.05 84.87) (end 146.05 87.63) (width 0.25) (layer B.Cu) (net 17))
   (segment (start 137.79641 87.63) (end 137.478205 87.948205) (width 0.25) (layer F.Cu) (net 17))
-  (segment (start 165.735 96.52) (end 165.735 95.25) (width 0.25) (layer F.Cu) (net 17))
-  (segment (start 164.20501 98.04999) (end 165.735 96.52) (width 0.25) (layer F.Cu) (net 17))
-  (segment (start 101.927909 98.04999) (end 164.20501 98.04999) (width 0.25) (layer F.Cu) (net 17))
   (segment (start 98.425 93.345) (end 98.425 94.547081) (width 0.25) (layer F.Cu) (net 17))
-  (segment (start 98.425 94.547081) (end 101.927909 98.04999) (width 0.25) (layer F.Cu) (net 17))
   (segment (start 133.985 80.01) (end 133.985 83.82) (width 0.25) (layer B.Cu) (net 17))
   (segment (start 133.985 80.01) (end 135.255 80.01) (width 0.25) (layer B.Cu) (net 17))
@@
   (segment (start 134.62 87.63) (end 137.16 87.63) (width 0.25) (layer F.Cu) (net 17))
   (segment (start 133.985 86.995) (end 134.62 87.63) (width 0.25) (layer F.Cu) (net 17))
+  (segment (start 165.735 96.38137) (end 164.96137 97.155) (width 0.25) (layer F.Cu) (net 17))
+  (segment (start 165.735 95.25) (end 165.735 96.38137) (width 0.25) (layer F.Cu) (net 17))
+  (segment (start 164.96137 97.155) (end 133.985 97.155) (width 0.25) (layer F.Cu) (net 17))
+  (segment (start 133.985 97.155) (end 133.985 93.98) (width 0.25) (layer F.Cu) (net 17))
+  (via (at 133.985 93.98) (size 0.8) (drill 0.4) (layers F.Cu B.Cu) (net 17))
+  (segment (start 133.985 93.98) (end 133.985 91.44) (width 0.25) (layer B.Cu) (net 17))
+  (via (at 133.985 91.44) (size 0.8) (drill 0.4) (layers F.Cu B.Cu) (net 17))
+  (segment (start 133.985 91.44) (end 133.985 86.995) (width 0.25) (layer F.Cu) (net 17))
   (segment (start 98.425 90.805) (end 101.6 90.805) (width 0.25) (layer F.Cu) (net 18))
   (segment (start 107.95 84.455) (end 107.95 74.93) (width 0.25) (layer F.Cu) (net 18))

Commit message: Add files via upload
Routing:
- net Net-(R2-Pad2): track 24.3 -> 25.8 mm
Changed lines of the file:
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@@
     (thickness 1.6)
     (drawings 15)
-    (tracks 201)
+    (tracks 202)
     (zones 0)
     (modules 20)
@@
   (segment (start 144.78 79.375) (end 147.955 82.55) (width 0.25) (layer B.Cu) (net 12))
   (segment (start 143.875 78.47) (end 144.78 79.375) (width 0.25) (layer B.Cu) (net 12))
-  (segment (start 124.939999 83.975001) (end 112.550001 83.975001) (width 0.25) (layer F.Cu) (net 13))
-  (segment (start 126.365 82.55) (end 124.939999 83.975001) (width 0.25) (layer F.Cu) (net 13))
-  (segment (start 110.49 81.915) (end 110.49 74.93) (width 0.25) (layer F.Cu) (net 13))
-  (segment (start 112.550001 83.975001) (end 110.49 81.915) (width 0.25) (layer F.Cu) (net 13))
+  (segment (start 125.095 84.95137) (end 126.365 83.68137) (width 0.25) (layer F.Cu) (net 13))
+  (segment (start 126.365 83.68137) (end 126.365 82.55) (width 0.25) (layer F.Cu) (net 13))
+  (segment (start 113.52637 84.95137) (end 125.095 84.95137) (width 0.25) (layer F.Cu) (net 13))
+  (segment (start 110.49 74.93) (end 110.49 81.915) (width 0.25) (layer F.Cu) (net 13))
+  (segment (start 110.49 81.915) (end 113.52637 84.95137) (width 0.25) (layer F.Cu) (net 13))
   (segment (start 115.57 50.82) (end 116.84 49.55) (width 0.25) (layer B.Cu) (net 14))
   (segment (start 115.57 52.07) (end 115.57 50.82) (width 0.25) (layer B.Cu) (net 14))

Commit message: Add files via upload
Routing:
- net +5V: track 168.3 -> 167.1 mm
Changed lines of the file:
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@@
     (thickness 1.6)
     (drawings 15)
-    (tracks 202)
+    (tracks 201)
     (zones 0)
     (modules 20)
@@
   (segment (start 146.05 84.87) (end 146.05 87.63) (width 0.25) (layer B.Cu) (net 17))
   (segment (start 137.79641 87.63) (end 137.478205 87.948205) (width 0.25) (layer F.Cu) (net 17))
-  (segment (start 98.425 93.345) (end 98.425 94.547081) (width 0.25) (layer F.Cu) (net 17))
   (segment (start 133.985 80.01) (end 133.985 83.82) (width 0.25) (layer B.Cu) (net 17))
   (segment (start 133.985 80.01) (end 135.255 80.01) (width 0.25) (layer B.Cu) (net 17))

Commit message: Add files via upload
Parts:
- J1, J3, J4: footprint Connector_Wago:Wago_734-132_1x02_P3.50mm_Vertical -> TerminalBlock:TerminalBlock_bornier-2_P5.08mm
- Q1, Q3: footprint Package_TO_SOT_THT:TO-92_Inline -> Package_TO_SOT_THT:TO-92_HandSolder
- Q2, Q4: footprint Package_TO_SOT_THT:TO-92_Inline -> Package_TO_SOT_THT:TO-92L_HandSolder
Routing:
- net Net-(J4-Pad1): track 25.9 -> 29.5 mm
- net GND: track 146.4 -> 149.3 mm
- net Net-(Q4-Pad2): track 12.5 -> 14.3 mm
- net Net-(Q2-Pad2): track 5.98 -> 4.71 mm
- net Net-(D2-Pad2): track 38.3 -> 37.1 mm
- net Net-(Q3-Pad2): track 18.5 -> 19.7 mm
Other:
- board text added: "Chain Counter WLAN Rev 1.1"
- board text removed: "Chain Counter WLAN Rev 1.0"

Commit message: Version 1.1
Parts:
- Q2, Q4: footprint Package_TO_SOT_THT:TO-92L_HandSolder -> Package_TO_SOT_THT:TO-92_HandSolder
Changed lines of the file:
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@@
+  )
+  (module Package_TO_SOT_THT:TO-92_HandSolder (layer F.Cu)
+    (at 137.16 76.835)
+    (descr "TO-92 leads molded, narrow, drill 0.75mm, handsoldering variant with enlarged pads (see NXP sot054_po.pdf)")
+    (tags "to-92 sc-43 sc-43a sot54 PA33 transistor")
+    (fp_text reference Q4 (at 1.27 -4.4) (layer F.SilkS)
+      (effects (font (size 1 1) (thickness 0.15)))
+    )
+    (fp_text value BC337 (at 1.27 2.79) (layer F.Fab)
+      (effects (font (size 1 1) (thickness 0.15)))
+    )
+    (fp_arc (start 1.27 0) (end 2.05 -2.45) (angle 117.6433766) (layer F.SilkS) (width 0.12))
+    (fp_arc (start 1.27 0) (end 1.27 -2.48) (angle -135) (layer F.Fab) (width 0.1))
+    (fp_arc (start 1.27 0) (end 0.45 -2.45) (angle -116.9632683) (layer F.SilkS) (width 0.12))
+    (fp_arc (start 1.27 0) (end 1.27 -2.48) (angle 135) (layer F.Fab) (width 0.1))
+    (fp_line (start 4 2.01) (end -1.46 2.01) (layer F.CrtYd) (width 0.05))
+    (fp_line (start 4 2.01) (end 4 -3.05) (layer F.CrtYd) (width 0.05))
+    (fp_line (start -1.45 -3.05) (end -1.46 2.01) (layer F.CrtYd) (width 0.05))
+    (fp_line (start -1.46 -3.05) (end 4 -3.05) (layer F.CrtYd) (width 0.05))
+    (fp_line (start -0.5 1.75) (end 3 1.75) (layer F.Fab) (width 0.1))
+    (fp_line (start -0.53 1.85) (end 3.07 1.85) (layer F.SilkS) (width 0.12))
+    (fp_text user %R (at 1.27 -4.4) (layer F.Fab)
+      (effects (font (size 1 1) (thickness 0.15)))
+    )
+    (pad 1 thru_hole rect (at 0 0) (size 1.1 1.8) (drill 0.75 (offset 0 0.4)) (layers *.Cu *.Mask)
+      (net 11 "Net-(Q4-Pad1)"))
+    (pad 3 thru_hole roundrect (at 2.54 0) (size 1.1 1.8) (drill 0.75 (offset 0 0.4)) (layers *.Cu *.Mask) (roundrect_rratio 0.25)
+      (net 18 GND))
+    (pad 2 thru_hole roundrect (at 1.27 -1.27) (size 1.1 1.8) (drill 0.75 (offset 0 -0.4)) (layers *.Cu *.Mask) (roundrect_rratio 0.25)
+      (net 12 "Net-(Q4-Pad2)"))
+    (model ${KISYS3DMOD}/Package_TO_SOT_THT.3dshapes/TO-92.wrl
+      (at (xyz 0 0 0))
+      (scale (xyz 1 1 1))
+      (rotate (xyz 0 0 0))
+    )
+  )
+  (module Package_TO_SOT_THT:TO-92_HandSolder (layer F.Cu)
+    (at 144.78 70.485)
+    (descr "TO-92 leads molded, narrow, drill 0.75mm, handsoldering variant with enlarged pads (see NXP sot054_po.pdf)")
+    (tags "to-92 sc-43 sc-43a sot54 PA33 transistor")
+    (fp_text reference Q2 (at 1.27 -4.4) (layer F.SilkS)
+      (effects (font (size 1 1) (thickness 0.15)))
+    )
+    (fp_text value BC337 (at 1.27 2.79) (layer F.Fab)
+      (effects (font (size 1 1) (thickness 0.15)))
+    )
+    (fp_arc (start 1.27 0) (end 2.05 -2.45) (angle 117.6433766) (layer F.SilkS) (width 0.12))
+    (fp_arc (start 1.27 0) (end 1.27 -2.48) (angle -135) (layer F.Fab) (width 0.1))
+    (fp_arc (start 1.27 0) (end 0.45 -2.45) (angle -116.9632683) (layer F.SilkS) (width 0.12))
+    (fp_arc (start 1.27 0) (end 1.27 -2.48) (angle 135) (layer F.Fab) (width 0.1))
+    (fp_line (start 4 2.01) (end -1.46 2.01) (layer F.CrtYd) (width 0.05))
+    (fp_line (start 4 2.01) (end 4 -3.05) (layer F.CrtYd) (width 0.05))
+    (fp_line (start -1.45 -3.05) (end -1.46 2.01) (layer F.CrtYd) (width 0.05))
+    (fp_line (start -1.46 -3.05) (end 4 -3.05) (layer F.CrtYd) (width 0.05))
+    (fp_line (start -0.5 1.75) (end 3 1.75) (layer F.Fab) (width 0.1))
+    (fp_line (start -0.53 1.85) (end 3.07 1.85) (layer F.SilkS) (width 0.12))
+    (fp_text user %R (at 1.27 -4.4) (layer F.Fab)
+      (effects (font (size 1 1) (thickness 0.15)))
+    )
+    (pad 1 thru_hole rect (at 0 0) (size 1.1 1.8) (drill 0.75 (offset 0 0.4)) (layers *.Cu *.Mask)
+      (net 3 "Net-(D3-Pad2)"))
+    (pad 3 thru_hole roundrect (at 2.54 0) (size 1.1 1.8) (drill 0.75 (offset 0 0.4)) (layers *.Cu *.Mask) (roundrect_rratio 0.25)
+      (net 18 GND))
+    (pad 2 thru_hole roundrect (at 1.27 -1.27) (size 1.1 1.8) (drill 0.75 (offset 0 -0.4)) (layers *.Cu *.Mask) (roundrect_rratio 0.25)
+      (net 8 "Net-(Q2-Pad2)"))
+    (model ${KISYS3DMOD}/Package_TO_SOT_THT.3dshapes/TO-92.wrl
+      (at (xyz 0 0 0))
+      (scale (xyz 1 1 1))
+      (rotate (xyz 0 0 0))
+    )
   )
   (module Package_TO_SOT_THT:TO-92_HandSolder (layer F.Cu)
@@
       (at (xyz 0 0 0))
       (scale (xyz 1 1 1))
-      (rotate (xyz 0 0 0))
-    )
-  )
-  (module Package_TO_SOT_THT:TO-92L_HandSolder (layer F.Cu)
-    (at 137.16 76.835)
-    (descr "TO-92L leads in-line (large body variant of TO-92), also known as TO-226, wide, drill 0.75mm, hand-soldering variant with enlarged pads (see https://www.diodes.com/assets/Package-Files/TO92L.pdf and http://www.ti.com/lit/an/snoa059/snoa059.pdf)")
-    (tags "to-92 sc-43 sc-43a sot54 PA33 transistor")
-    (fp_text reference Q4 (at 1.27 -3.8) (layer F.SilkS)
-      (effects (font (size 1 1) (thickness 0.15)))
-    )
-    (fp_text value BC337 (at 1.27 2.79) (layer F.Fab)
-      (effects (font (size 1 1) (thickness 0.15)))
-    )
-    (fp_arc (start 1.27 0) (end 2.05 -2.45) (angle 117.6433766) (layer F.SilkS) (width 0.12))
-    (fp_arc (start 1.27 0) (end 1.27 -2.48) (angle -135) (layer F.Fab) (width 0.1))
-    (fp_arc (start 1.27 0) (end 0.45 -2.45) (angle -116.9763941) (layer F.SilkS) (width 0.12))
-    (fp_arc (start 1.27 0) (end 1.27 -2.48) (angle 135) (layer F.Fab) (width 0.1))
-    (fp_line (start 4 2.01) (end -1.46 2.01) (layer F.CrtYd) (width 0.05))
-    (fp_line (start 4 2.01) (end 4 -3.05) (layer F.CrtYd) (width 0.05))
-    (fp_line (start -1.45 -3.05) (end -1.46 2.01) (layer F.CrtYd) (width 0.05))
-    (fp_line (start -1.46 -3.05) (end 4 -3.05) (layer F.CrtYd) (width 0.05))
-    (fp_line (start -0.5 1.75) (end 3 1.75) (layer F.Fab) (width 0.1))
-    (fp_line (start -0.53 1.85) (end 3.07 1.85) (layer F.SilkS) (width 0.12))
-    (fp_text user %R (at 1.27 0) (layer F.Fab)
-      (effects (font (size 1 1) (thickness 0.15)))
-    )
-    (pad 1 thru_hole rect (at 0 0) (size 1.1 1.8) (drill 0.75 (offset 0 0.4)) (layers *.Cu *.Mask)
-      (net 11 "Net-(Q4-Pad1)"))
-    (pad 3 thru_hole roundrect (at 2.54 0) (size 1.1 1.8) (drill 0.75 (offset 0 0.4)) (layers *.Cu *.Mask) (roundrect_rratio 0.25)
-      (net 18 GND))
-    (pad 2 thru_hole roundrect (at 1.27 -1.27) (size 1.1 1.8) (drill 0.75 (offset 0 -0.4)) (layers *.Cu *.Mask) (roundrect_rratio 0.25)
-      (net 12 "Net-(Q4-Pad2)"))
-    (model ${KISYS3DMOD}/Package_TO_SOT_THT.3dshapes/TO-92L.wrl
-      (at (xyz 0 0 0))
-      (scale (xyz 1 1 1))
-      (rotate (xyz 0 0 0))
-    )
-  )
-  (module Package_TO_SOT_THT:TO-92L_HandSolder (layer F.Cu)
-    (at 144.78 70.485)
-    (descr "TO-92L leads in-line (large body variant of TO-92), also known as TO-226, wide, drill 0.75mm, hand-soldering variant with enlarged pads (see https://www.diodes.com/assets/Package-Files/TO92L.pdf and http://www.ti.com/lit/an/snoa059/snoa059.pdf)")
-    (tags "to-92 sc-43 sc-43a sot54 PA33 transistor")
-    (fp_text reference Q2 (at 1.27 -3.8) (layer F.SilkS)
-      (effects (font (size 1 1) (thickness 0.15)))
-    )
-    (fp_text value BC337 (at 1.27 2.79) (layer F.Fab)
-      (effects (font (size 1 1) (thickness 0.15)))
-    )
-    (fp_arc (start 1.27 0) (end 2.05 -2.45) (angle 117.6433766) (layer F.SilkS) (width 0.12))
-    (fp_arc (start 1.27 0) (end 1.27 -2.48) (angle -135) (layer F.Fab) (width 0.1))
-    (fp_arc (start 1.27 0) (end 0.45 -2.45) (angle -116.9763941) (layer F.SilkS) (width 0.12))
-    (fp_arc (start 1.27 0) (end 1.27 -2.48) (angle 135) (layer F.Fab) (width 0.1))
-    (fp_line (start 4 2.01) (end -1.46 2.01) (layer F.CrtYd) (width 0.05))
-    (fp_line (start 4 2.01) (end 4 -3.05) (layer F.CrtYd) (width 0.05))
-    (fp_line (start -1.45 -3.05) (end -1.46 2.01) (layer F.CrtYd) (width 0.05))
-    (fp_line (start -1.46 -3.05) (end 4 -3.05) (layer F.CrtYd) (width 0.05))
-    (fp_line (start -0.5 1.75) (end 3 1.75) (layer F.Fab) (width 0.1))
-    (fp_line (start -0.53 1.85) (end 3.07 1.85) (layer F.SilkS) (width 0.12))
-    (fp_text user %R (at 1.27 0) (layer F.Fab)
-      (effects (font (size 1 1) (thickness 0.15)))
-    )
-    (pad 1 thru_hole rect (at 0 0) (size 1.1 1.8) (drill 0.75 (offset 0 0.4)) (layers *.Cu *.Mask)
-      (net 3 "Net-(D3-Pad2)"))
-    (pad 3 thru_hole roundrect (at 2.54 0) (size 1.1 1.8) (drill 0.75 (offset 0 0.4)) (layers *.Cu *.Mask) (roundrect_rratio 0.25)
-      (net 18 GND))
-    (pad 2 thru_hole roundrect (at 1.27 -1.27) (size 1.1 1.8) (drill 0.75 (offset 0 -0.4)) (layers *.Cu *.Mask) (roundrect_rratio 0.25)
-      (net 8 "Net-(Q2-Pad2)"))
-    (model ${KISYS3DMOD}/Package_TO_SOT_THT.3dshapes/TO-92L.wrl
-      (at (xyz 0 0 0))
-      (scale (xyz 1 1 1))
